Commit message: update: changed the camera setting

File: lgmcts/assets/ur5/workspace.urdf (robot description, URDF)
Before this commit: robot workspace.urdf, 1 links, 0 joints
Links:
- link baseLink: geometry visual mesh filename=plane.obj scale=0.0333 0.0333 1

Commit message: update: fix the collision in 90 percent

File: lgmcts/assets/ur5/workspace.urdf (robot description, URDF)
Before this commit: robot workspace.urdf, 1 links, 0 joints
Links:
- link baseLink: geometry visual mesh filename=plane.obj scale=0.0167 0.0333 1
